File: hardware/V2/esp32_master_board.sch (EAGLE design)
At the start: 62 parts, among them IC1 SN74HC138PW, IC2 MAX17502EATB+T, IC3 WS2812B, IC4 WS2812B, SW1 B3U-1000P-2P-SMD

Commit message: update BOM, correct C2 and R17 MPN; remove deprecated seeed BOM
Parts:
- C2: MANUFACTURER_PART_NUMBER 0101ZC471KAT2A -> CL05C471JB5NNNC
- R17: MANUFACTURER_PART_NUMBER CPL-RES-0603-1.5K-0.1W -> ERJ2GEJ152X
Changed lines of the file:
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@@
 <?xml version="1.0" encoding="utf-8"?>
 <!DOCTYPE eagle SYSTEM "eagle.dtd">
-<eagle version="9.5.0">
+<eagle version="9.6.2">
 <drawing>
 <settings>
@@
 <part name="P+2" library="supply1" library_urn="urn:adsk.eagle:library:371" deviceset="VCC" device=""/>
 <part name="C2" library="resistor" library_urn="urn:adsk.eagle:library:348" deviceset="C-EU" device="C0402" package3d_urn="urn:adsk.eagle:package:23626/2" value="470p">
-<attribute name="MANUFACTURER_PART_NUMBER" value="0101ZC471KAT2A"/>
+<attribute name="MANUFACTURER_PART_NUMBER" value="CL05C471JB5NNNC"/>
 </part>
 <part name="C3" library="resistor" library_urn="urn:adsk.eagle:library:348" deviceset="C-EU" device="C0402" package3d_urn="urn:adsk.eagle:package:23626/2" value="1u LOW ESR">
@@
 <part name="P+4" library="supply1" library_urn="urn:adsk.eagle:library:371" deviceset="VCC" device=""/>
 <part name="R17" library="resistor" library_urn="urn:adsk.eagle:library:348" deviceset="R-EU_" device="R0402" package3d_urn="urn:adsk.eagle:package:26058/2" value="1.5k">
-<attribute name="MANUFACTURER_PART_NUMBER" value="CPL-RES-0603-1.5K-0.1W"/>
+<attribute name="MANUFACTURER_PART_NUMBER" value="ERJ2GEJ152X"/>
 </part>
 <part name="P+6" library="supply1" library_urn="urn:adsk.eagle:library:371" deviceset="VCC" device=""/>

Commit message: Fix 0402 footprint to comply with seeed, fix HR911105A footprint, add labels for L1,U,U,U,U, update board revision to V2.2
Parts:
- U$3: device HR911105A:HR911105A -> HR911105A_bis:HR911105A
Connections:
- net GND: now also U$3.SHIELD; no longer U$3.SHIELD0, U$3.SHIELD1
- net N$11: now also U$3.YC; no longer U$3.Y-
- net N$12: now also U$3.GC; no longer U$3.G-
- net VDD: now also U$3.GA, U$3.YA; no longer U$3.G+, U$3.Y+
Other:
- note added: "MASTER BOARD V2.2 LAAS CNRS - Thomas FLAYOLS https://github.com/open-dynamic-robot-initiative/master-board"
- note removed: "MASTER BOARD V2.1 LAAS CNRS - Thomas FLAYOLS https://github.com/open-dynamic-robot-initiative/master-board"
- moved on the sheet: C1, C5, C6, R8, R9
